File: bpf-tun.kicad_sch (KiCad schematic)
At the start: 44 parts

Commit message: 部品定数を入力　ただし未評価
Parts:
- C501, C502, C529, C530: value 10p -> NM
- C503, C505, C507, C509, C511, C513, C515, C517, C519, C521, C523, C525, C527: value 1p -> NM
- L503, L505: value 10n -> NM
- L504, L506: value 1u -> 10n
Other:
- note added: "8.0mm 鉛筆に0.5mmを巻く 3.5mm 3.2mmドリルに0.5mmを巻く"
- note added: "Not Mount(for testing)"
- note added: "filter https://rf-tools.com/lc-filter/ coil http://gate.ruru.ne.jp/rfdn/Tools/ScoilForm.asp"
- note added: "トリマ 青 5p 白 10p 赤 20p 緑 30p 黄 40pトリマ 青 5p 白 10p 赤 20p 緑 30p 黄 40p"
- company: (none) -> JK1MLY / PRUG
- title: (none) -> FM QRP TRCV
