File: main.kicad_sch (KiCad schematic)
At the start: 63 parts, among them IC11 PIC16F1503T-I/SL, IC12 BK4802P, IC12 LM2940T-3.3, IC13 NJM2391DL1-33, J11 Conn_01x03, J12 Conn_01x06, J13 Conn_01x03, J14 Conn_Coaxial, J15 Conn_01x03, J16 Conn_01x03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

Commit message: Add files via upload
Parts:
- C20: value 1u -> 0.1u
- C22, C24: value 0.1u -> 1u
- C23: value 30p -> 10p
- renumbered IC12 to IC13, IC13 to U12
Other:
- note added: "12Vの場合はレギュレータの放熱に注意 3.3V供給とする場合はU11でジャンパ"
- note added: "R17はカイロミス 本来は3.3Vラインの切り離し用"
- note added: "ダイオードスイッチ用"
- note removed: "12Vの場合はレギュレータの放熱に注意 3.3V供給とする場合はジャンパ"
- note removed: "周波数制御のサンプルプログラム https://github.com/jk1mly/fm-trcv 参考 BG7QKU https://github.com/BG7QKU BK4802N https://aitendo3.sakura.ne.jp/aitendo_data/product_img/ic/wirless/BK4802P/BK4802N-BEKEN.pdf"
- note removed: "基本的にフィルタは外付"
- note removed: "外部に送受信のアンプを追加 バンドパスフィルタを追加する 場合の制御用"
- moved on the sheet: TP1, TP2, TP3, TP4, TP5
