File: fm_qrp2.kicad_pcb (KiCad board)
At the start: 2 copper layers, 100 x 80 mm, 153 parts, among them IC11 PIC16F1503T-I/SL, IC12 BK4802P, J11 Conn_01x03, J12 Conn_01x06, J13 Conn_01x03, J14 Conn_Coaxial, J15 Conn_01x03, J16 Conn_01x03, J17 Conn_01x03, J18 Conn_01x04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

Commit message: アップデート
Parts:
- removed C301, C312, C401, C412: NM, Capacitor_THT:C_Disc_D3.4mm_W2.1mm_P2.50mm
- removed C308, C408: 4p, Capacitor_THT:C_Disc_D3.4mm_W2.1mm_P2.50mm
- removed SW11: SW_SPDT, digikey-footprints:Switch_Slide_11.6x4mm_EG1218
- added ?: , , F.Cu at (157.6, 98.7)
- added ?: , , F.Cu at (173.9, 110.7)
- added ?: , , F.Cu at (173.9, 98.8)
- added ?: , , F.Cu at (157.6, 110.7)
- added ?: , , F.Cu at (154.3, 69.2)
- added ?: , , F.Cu at (177.2, 80.6)
- added ?: , , F.Cu at (177.2, 69.8)
- added ?: , , F.Cu at (154.6, 80.6)
- added C11: 470u, Capacitor_THT:CP_Radial_D7.5mm_P2.50mm, F.Cu at (196.2, 125.1)
- added C31: 0.1u, Capacitor_THT:C_Disc_D3.4mm_W2.1mm_P2.50mm, F.Cu at (193.7, 74.0)
- added C32: 0.1u, Capacitor_THT:C_Disc_D3.4mm_W2.1mm_P2.50mm, F.Cu at (196.2, 97.3)
- added D14: LED, digikey-footprints:LED_3mm_Radial, F.Cu at (140.3, 115.6)
- added R105: 1k, Resistor_THT:R_Axial_DIN0207_L6.3mm_D2.5mm_P2.54mm_Vertical, F.Cu at (188.6, 69.2)
- added R205: 1k, Resistor_THT:R_Axial_DIN0207_L6.3mm_D2.5mm_P2.54mm_Vertical, F.Cu at (186.1, 89.5)
- added R24: 1k, Resistor_THT:R_Axial_DIN0207_L6.3mm_D2.5mm_P2.54mm_Vertical, F.Cu at (135.3, 115.6)
- added R305: 1k, Resistor_THT:R_Axial_DIN0207_L6.3mm_D2.5mm_P2.54mm_Vertical, F.Cu at (191.1, 99.7)
- added R405: 1k, Resistor_THT:R_Axial_DIN0207_L6.3mm_D2.5mm_P2.54mm_Vertical, F.Cu at (183.5, 115.1)
- added TP12: TestPoint, Connector_PinHeader_2.54mm:PinHeader_1x01_P2.54mm_Vertical, F.Cu at (133.3, 104.1)
- C15: footprint Capacitor_THT:CP_Radial_Tantal_D7.0mm_P2.50mm -> Capacitor_THT:CP_Radial_D7.5mm_P2.50mm
- C26: value 1000p -> 0.01u
- C29: footprint Capacitor_THT:CP_Radial_Tantal_D5.0mm_P2.50mm -> Capacitor_THT:CP_Radial_D5.0mm_P2.00mm
- C304, C309: value 10p -> 15p
- C305: value NM -> 15p
- C306: value 4p -> 33p
- C307: value 22p -> 15p
- D101, D102, D201, D202, D301, D302, D401, D402: footprint Diode_THT:D_A-405_P2.54mm_Vertical_AnodeUp -> Diode_THT:D_T-1_P5.08mm_Horizontal
- D11: footprint Diode_THT:D_DO-41_SOD81_P10.16mm_Horizontal -> Diode_THT:D_DO-34_SOD68_P7.62mm_Horizontal
- R15, R20: footprint Resistor_THT:R_Axial_DIN0204_L3.6mm_D1.6mm_P7.62mm_Horizontal -> Resistor_THT:R_Axial_DIN0207_L6.3mm_D2.5mm_P2.54mm_Vertical
- R21: footprint Resistor_THT:R_Axial_DIN0207_L6.3mm_D2.5mm_P2.54mm_Vertical -> Resistor_THT:R_Axial_DIN0204_L3.6mm_D1.6mm_P7.62mm_Horizontal
- moved C30 29.6 mm to (130.2, 112.4), turned to 0 degrees
- moved R22 16.5 mm to (130.2, 132.7), turned to 90 degrees
- moved R21 15.5 mm to (122.6, 117.5), turned to -90 degrees
- moved C402 15.4 mm to (142.9, 89.6), turned to -90 degrees
- moved D11 15.2 mm to (191.1, 122.6), turned to 180 degrees
- moved L401 11.3 mm to (140.3, 97.3)
- moved R15 10.8 mm to (135.3, 132.7), turned to 0 degrees
- moved R103 10.7 mm to (188.6, 71.6)
- moved Q14 10.2 mm to (137.8, 94.6), turned to 90 degrees
- moved L106 9.20 mm to (191.1, 74.1)
- moved L402 9.14 mm to (142.9, 104.8), turned to -90 degrees
- moved D102 9.12 mm to (191.1, 76.8)
- moved D401 8.07 mm to (142.9, 97.2), turned to -90 degrees
- moved R402 8.04 mm to (145.4, 112.4)
- moved J17 8.03 mm to (132.7, 125.1), turned to 0 degrees
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- renumbered C11 to C33, U13 to IC13
Connections:
- IC11 pad 5: unconnected-(IC11-PWM1/CLC1/CWG1A/RC5-Pad5) -> Net-(IC11-PWM1/CLC1/CWG1A/RC5)
- J11 pad 1: Net-(J11-Pin_1) -> /RF-IC/+5VIN
- L304 pad 1: Net-(C308-Pad2) -> Net-(C306-Pad2)
- L404 pad 1: Net-(C408-Pad2) -> Net-(C406-Pad2)
- R103 pad 1: Net-(L105-Pad2) -> +5V
- R103 pad 2: +5V -> Net-(L105-Pad2)
- R20 pad 1: Net-(D13-K) -> GND
- R20 pad 2: GND -> Net-(D13-K)
Routing:
- net GND: track 614.3 -> 358.0 mm, vias 119 -> 133
- net +3V3: track 77.3 -> 98.0 mm
- net +5V: track 240.3 -> 256.6 mm
- net RFIO: track 35.2 -> 19.9 mm
- net Net-(IC11-RA3/T1G/CLC1IN0/~{SS}/~{MCLR}/Vpp): track 25.0 -> 39.9 mm, vias 0 -> 1
- net RFANT: track 36.5 -> 25.2 mm
- net /RF-IC/+5VIN: track 29.4 -> 40.2 mm
- net Net-(J12-Pin_2): track 15.4 -> 5.08 mm
- net Net-(J11-Pin_1): track 10.1 -> 0.00 mm
- net Net-(D12-A): track 13.5 -> 4.60 mm
- net Net-(IC11-PWM1/CLC1/CWG1A/RC5): track 0.00 -> 8.52 mm
- net Net-(D14-A): track 44.3 -> 36.4 mm, vias 0 -> 2
- net B28: track 63.1 -> 55.4 mm
- net Net-(D101-K): track 14.8 -> 7.60 mm
- net Net-(IC11-CLC2IN1/CWG1B/C2OUT/RC4): track 15.9 -> 22.6 mm
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Other:
- board text added: "+"
- board text added: "21M25"
- board text added: "4.95 3.5-3.5"
- board text added: "6.37mm"
- board text added: "JK1MLY 2023.7"
- board text added: "RC5"
- board text removed: "EAR+"
- board text removed: "JK1MLY 2023.6"
- board text removed: "SPK+"
- board text removed: "SPK-"

Commit message: Add files via upload
Changed lines of the file:
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@@
     (property "ki_keywords" "cap capacitor")
     (attr through_hole)
-    (fp_text reference "C302" (at 2.5 2.58 90) (layer "F.SilkS") hide
+    (fp_text reference "C302" (at -2.555 6.1 90) (layer "F.SilkS")
         (effects (font (size 1 1) (thickness 0.15)))
     )
@@
   (gr_line (start 151.13 93.345) (end 154.305 93.345)
     (stroke (width 0.12) (type default)) (layer "F.SilkS"))
+  (gr_line (start 140.315 87.63) (end 143.8 88.985)
+    (stroke (width 0.12) (type default)) (layer "F.SilkS"))
   (gr_poly
